Commit message: formatted code

File: eufs_description/urdf/bases/ads-dv_base.urdf.xacro (robot description, xacro)
@@ -3,19 +3,19 @@
   <xacro:include filename="$(find eufs_description)/urdf/bases/eufs_base.gazebo.xacro" />
   <xacro:macro name="eufs_base" params="name publish_bf hq">
-  <!-- Robot mechanical and motor parameters -->
-  <xacro:property name="PI" value="3.1415926535897931"/>
-  <xacro:property name="wheel_width" value="0.175" />
-  <!-- <xacro:property name="clearance" value="${tire_dia/2.0}" /> -->
-  <xacro:property name="clearance" value="0.25" />
-  <!-- BASE FOOTPRINT -->
-  <xacro:if value="${publish_bf}">
-    <link name="base_footprint">
-      <visual>
+    <!-- Robot mechanical and motor parameters -->
+    <xacro:property name="PI" value="3.1415926535897931" />
+    <xacro:property name="wheel_width" value="0.175" />
+    <!-- <xacro:property name="clearance" value="${tire_dia/2.0}" /> -->
+    <xacro:property name="clearance" value="0.25" />
+    <!-- BASE FOOTPRINT -->
+    <xacro:if value="${publish_bf}">
+      <link name="base_footprint">
+        <visual>
           <origin xyz="0 0 0" rpy="0 0 0" />
           <geometry>
-             <box size="0.001 0.001 0.001" />
+            <box size="0.001 0.001 0.001" />
           </geometry>
-      </visual>
-<!--
+        </visual>
+        <!--
       <collision>
           <origin xyz="0 0 0" rpy="0 0 0" />
@@ -25,56 +25,56 @@
       </collision>
 -->
+      </link>
+      <joint name="base_footprint_joint" type="fixed">
+        <origin xyz="0 0 ${clearance}" rpy="0 0 0" /> <!-- height is the clearance -->
+        <parent link="base_footprint" />
+        <child link="base_link" />
+      </joint>
+    </xacro:if>
+    <!-- BASE_LINK -->
+    <link name="base_link">
+      <inertial>
+        <mass value="125.0" />
+        <origin xyz="0 0 0" />
+        <inertia ixx="1.391" ixy="0.004" ixz="0.0" iyy="6.853" iyz="0.0" izz="6.125" />
+      </inertial>
+      <visual>
+        <origin xyz="0 0 0" rpy="0 0 0" />
+        <xacro:if value="${hq}">
+          <geometry>
+            <mesh filename="package://eufs_description/meshes/ads-dv.dae" />
+          </geometry>
+        </xacro:if>
+        <xacro:unless value="${hq}">
+          <geometry>
+            <mesh filename="package://eufs_description/meshes/ads-dv.dae" />
+          </geometry>
+        </xacro:unless>
+      </visual>
+      <collision>
+        <origin xyz="0 0 0" rpy="0 0 0 " />
+        <geometry>
+          <mesh filename="package://eufs_description/meshes/ads-dv.dae" />
+        </geometry>
+      </collision>
     </link>
-    <joint name="base_footprint_joint" type="fixed">
-      <origin xyz="0 0 ${clearance}" rpy="0 0 0" />  <!-- height is the clearance -->
-      <parent link="base_footprint"/>
-      <child link="base_link" />
+    <link name="odom_ground_truth">
+      <collision>
+        <geometry>
+          <box size="0.1 0.1 0.1" />
+        </geometry>
+      </collision>
+      <inertial>
+        <mass value="1e-5" />
+        <origin xyz="0 0 0" rpy="0 0 0" />
+        <inertia ixx="1e-6" ixy="0" ixz="0" iyy="1e-6" iyz="0" izz="1e-6" />
+      </inertial>
+    </link>
+    <joint name="odom_ground_truth_joint" type="fixed">
+      <axis xyz="0 0 0" />
+      <origin xyz="0 0 0" rpy="0 0 0" />
+      <parent link="base_link" />
+      <child link="odom_ground_truth" />
     </joint>
-  </xacro:if>
-  <!-- BASE_LINK -->
-  <link name="base_link">
-    <inertial>
-      <mass value="125.0" />
-      <origin xyz="0 0 0" />
-      <inertia  ixx="1.391" ixy="0.004"  ixz="0.0"  iyy="6.853"  iyz="0.0"  izz="6.125" />
-    </inertial>
-    <visual>
-       <origin xyz="0 0 0" rpy="0 0 0" />
-       <xacro:if value="${hq}">
-       <geometry>
-	     <mesh filename="package://eufs_description/meshes/ads-dv.dae"/>
-       </geometry>
-       </xacro:if>
-       <xacro:unless value="${hq}">
-       <geometry>
-	     <mesh filename="package://eufs_description/meshes/ads-dv.dae"/>
-       </geometry>
-       </xacro:unless>
-    </visual>
-    <collision>
-       <origin xyz="0 0 0" rpy="0 0 0 " />
-       <geometry>
-         <mesh filename="package://eufs_description/meshes/ads-dv.dae"/>
-       </geometry>
-    </collision>
-  </link>
-  <link name="odom_ground_truth">
-    <collision>
-      <geometry>
-        <box size="0.1 0.1 0.1"/>
-      </geometry>
-    </collision>
-    <inertial>
-      <mass value="1e-5" />
-      <origin xyz="0 0 0" rpy="0 0 0"/>
-      <inertia ixx="1e-6" ixy="0" ixz="0" iyy="1e-6" iyz="0" izz="1e-6" />
-    </inertial>
-  </link>
-  <joint name="odom_ground_truth_joint" type="fixed">
-    <axis xyz="0 0 0" />
-    <origin xyz="0 0 0" rpy="0 0 0"/>
-    <parent link="base_link"/>
-    <child link="odom_ground_truth"/>
-  </joint>
   </xacro:macro>
 </robot>

File: eufs_description/urdf/bases/eufs_base.gazebo.xacro (robot description, xacro)
@@ -9,19 +9,19 @@
         <!-- controlPeriod>0.003</controlPeriod -->
         <controlPeriod>0.001</controlPeriod>
-	    <robotSimType>gazebo_ros_control/DefaultRobotHWSim</robotSimType>
+        <robotSimType>gazebo_ros_control/DefaultRobotHWSim</robotSimType>
       </plugin>
     </gazebo>
-	</xacro:macro>
+  </xacro:macro>
   <gazebo>
     <plugin name="p3d_base_controller" filename="libgazebo_ros_p3d.so">
-        <alwaysOn>true</alwaysOn>
-        <updateRate>200.0</updateRate>
-        <bodyName>odom_ground_truth</bodyName>
-        <topicName>ground_truth/state_raw</topicName>
-        <gaussianNoise>0.00</gaussianNoise>
-        <frameName>world</frameName>
-        <!-- origin is at spawn location -->
-        <xyzOffset>43.0 -40 0</xyzOffset>
-        <rpyOffset>0 0 0</rpyOffset>
+      <alwaysOn>true</alwaysOn>
+      <updateRate>200.0</updateRate>
+      <bodyName>odom_ground_truth</bodyName>
+      <topicName>ground_truth/state_raw</topicName>
+      <gaussianNoise>0.00</gaussianNoise>
+      <frameName>world</frameName>
+      <!-- origin is at spawn location -->
+      <xyzOffset>43.0 -40 0</xyzOffset>
+      <rpyOffset>0 0 0</rpyOffset>
     </plugin>
   </gazebo>

File: eufs_description/urdf/bases/eufs_base.urdf.xacro (robot description, xacro)
@@ -3,19 +3,19 @@
   <xacro:include filename="$(find eufs_description)/urdf/bases/eufs_base.gazebo.xacro" />
   <xacro:macro name="eufs_base" params="name publish_bf hq">
-  <!-- Robot mechanical and motor parameters -->
-  <xacro:property name="PI" value="3.1415926535897931"/>
-  <xacro:property name="wheel_width" value="0.175" />
-  <!-- <xacro:property name="clearance" value="${tire_dia/2.0}" /> -->
-  <xacro:property name="clearance" value="0.25" />
-  <!-- BASE FOOTPRINT -->
-  <xacro:if value="${publish_bf}">
-    <link name="base_footprint">
-      <visual>
+    <!-- Robot mechanical and motor parameters -->
+    <xacro:property name="PI" value="3.1415926535897931" />
+    <xacro:property name="wheel_width" value="0.175" />
+    <!-- <xacro:property name="clearance" value="${tire_dia/2.0}" /> -->
+    <xacro:property name="clearance" value="0.25" />
+    <!-- BASE FOOTPRINT -->
+    <xacro:if value="${publish_bf}">
+      <link name="base_footprint">
+        <visual>
           <origin xyz="0 0 0" rpy="0 0 0" />
           <geometry>
-             <box size="0.001 0.001 0.001" />
+            <box size="0.001 0.001 0.001" />
           </geometry>
-      </visual>
-<!--
+        </visual>
+        <!--
       <collision>
           <origin xyz="0 0 0" rpy="0 0 0" />
@@ -25,56 +25,56 @@
       </collision>
 -->
+      </link>
+      <joint name="base_footprint_joint" type="fixed">
+        <origin xyz="0 0 ${clearance}" rpy="0 0 0" /> <!-- height is the clearance -->
+        <parent link="base_footprint" />
+        <child link="base_link" />
+      </joint>
+    </xacro:if>
+    <!-- BASE_LINK -->
+    <link name="base_link">
+      <inertial>
+        <mass value="125.0" />
+        <origin xyz="0 0 0" />
+        <inertia ixx="1.391" ixy="0.004" ixz="0.0" iyy="6.853" iyz="0.0" izz="6.125" />
+      </inertial>
+      <visual>
+        <origin xyz="0 0 0" rpy="0 0 0" />
+        <xacro:if value="${hq}">
+          <geometry>
+            <mesh filename="package://eufs_description/meshes/chassis.dae" />
+          </geometry>
+        </xacro:if>
+        <xacro:unless value="${hq}">
+          <geometry>
+            <mesh filename="package://eufs_description/meshes/chassis.dae" />
+          </geometry>
+        </xacro:unless>
+      </visual>
+      <collision>
+        <origin xyz="0 0 0" rpy="0 0 0 " />
+        <geometry>
+          <mesh filename="package://eufs_description/meshes/chassis_collision.dae" />
+        </geometry>
+      </collision>
     </link>
-    <joint name="base_footprint_joint" type="fixed">
-      <origin xyz="0 0 ${clearance}" rpy="0 0 0" />  <!-- height is the clearance -->
-      <parent link="base_footprint"/>
-      <child link="base_link" />
+    <link name="odom_ground_truth">
+      <collision>
+        <geometry>
+          <box size="0.1 0.1 0.1" />
+        </geometry>
+      </collision>
+      <inertial>
+        <mass value="1e-5" />
+        <origin xyz="0 0 0" rpy="0 0 0" />
+        <inertia ixx="1e-6" ixy="0" ixz="0" iyy="1e-6" iyz="0" izz="1e-6" />
+      </inertial>
+    </link>
+    <joint name="odom_ground_truth_joint" type="fixed">
+      <axis xyz="0 0 0" />
+      <origin xyz="0 0 0" rpy="0 0 0" />
+      <parent link="base_link" />
+      <child link="odom_ground_truth" />
     </joint>
-  </xacro:if>
-  <!-- BASE_LINK -->
-  <link name="base_link">
-    <inertial>
-      <mass value="125.0" />
-      <origin xyz="0 0 0" />
-      <inertia  ixx="1.391" ixy="0.004"  ixz="0.0"  iyy="6.853"  iyz="0.0"  izz="6.125" />
-    </inertial>
-    <visual>
-       <origin xyz="0 0 0" rpy="0 0 0" />
-       <xacro:if value="${hq}">
-       <geometry>
-	     <mesh filename="package://eufs_description/meshes/chassis.dae"/>
-       </geometry>
-       </xacro:if>
-       <xacro:unless value="${hq}">
-       <geometry>
-	     <mesh filename="package://eufs_description/meshes/chassis.dae"/>
-       </geometry>
-       </xacro:unless>
-    </visual>
-    <collision>
-       <origin xyz="0 0 0" rpy="0 0 0 " />
-       <geometry>
-         <mesh filename="package://eufs_description/meshes/chassis_collision.dae"/>
-       </geometry>
-    </collision>
-  </link>
-  <link name="odom_ground_truth">
-    <collision>
-      <geometry>
-        <box size="0.1 0.1 0.1"/>
-      </geometry>
-    </collision>
-    <inertial>
-      <mass value="1e-5" />
-      <origin xyz="0 0 0" rpy="0 0 0"/>
-      <inertia ixx="1e-6" ixy="0" ixz="0" iyy="1e-6" iyz="0" izz="1e-6" />
-    </inertial>
-  </link>
-  <joint name="odom_ground_truth_joint" type="fixed">
-    <axis xyz="0 0 0" />
-    <origin xyz="0 0 0" rpy="0 0 0"/>
-    <parent link="base_link"/>
-    <child link="odom_ground_truth"/>
-  </joint>
   </xacro:macro>
 </robot>
