Commit message: formatted code

File: eufs_description/urdf/wheels/suspension_wheel.urdf.xacro (robot description, xacro)
@@ -6,30 +6,30 @@
        is a "zero offset" wheel. hex_hub_depth = tire_width / 2 -
        axle_length. -->
-  <xacro:property name="hub_dia" value="0.08"/>
-  <xacro:property name="tire_dia" value="0.505"/>
-  <xacro:property name="tire_width" value="0.2"/>
-  <xacro:property name="hex_hub_depth" value="0.120"/> <!-- or +0.072 -->
-  <xacro:property name="wheel_mass" value="10.0"/>   <!-- check -->
+  <xacro:property name="hub_dia" value="0.08" />
+  <xacro:property name="tire_dia" value="0.505" />
+  <xacro:property name="tire_width" value="0.2" />
+  <xacro:property name="hex_hub_depth" value="0.120" /> <!-- or +0.072 -->
+  <xacro:property name="wheel_mass" value="10.0" /> <!-- check -->
   <!-- hex_hub_dist is the distance between left and right hex hubs when
        the shock absorbers are fully extended. axle_length is the distance
        from a U joint to the corresponding hex hub. wheel_travel is the
        vertical wheel travel. -->
-  <xacro:property name="wheelbase" value="1.55"/>
-  <xacro:property name="hex_hub_dist" value="1.360"/>  <!-- track/width of the car -->
-  <xacro:property name="axle_length" value="0.120"/>
-  <xacro:property name="wheel_travel" value="0.05"/>
-  <xacro:property name="shock_z_offset" value="0.05"/>
+  <xacro:property name="wheelbase" value="1.55" />
+  <xacro:property name="hex_hub_dist" value="1.360" /> <!-- track/width of the car -->
+  <xacro:property name="axle_length" value="0.120" />
+  <xacro:property name="wheel_travel" value="0.05" />
+  <xacro:property name="shock_z_offset" value="0.05" />
   <!-- Degree-to-radian conversions -->
-  <xacro:property name="degrees_45" value="0.785398163"/>
-  <xacro:property name="degrees_90" value="1.57079633"/>
-  <xacro:property name="degrees_180" value="3.14159265"/>
+  <xacro:property name="degrees_45" value="0.785398163" />
+  <xacro:property name="degrees_90" value="1.57079633" />
+  <xacro:property name="degrees_180" value="3.14159265" />
   <!-- shock_eff_limit is 2 * ((shock_stroke / 2) * shock_spring_constant) N. -->
-  <xacro:property name="shock_eff_limit" value="50"/>
-  <xacro:property name="shock_vel_limit" value="500"/>
+  <xacro:property name="shock_eff_limit" value="50" />
+  <xacro:property name="shock_vel_limit" value="500" />
   <xacro:property name="wheel_joint_damping" value="0.01" />
   <xacro:property name="wheel_joint_friction" value="0.1" />
   <xacro:property name="suspension_joint_damping" value="0.01" />
   <xacro:property name="suspension_joint_friction" value="0.1" />
-<!--          max_speed = 100mph = 44.704 m/s
+  <!--          max_speed = 100mph = 44.704 m/s
        axle_vel_limit = (2 * pi) * (max_speed / (pi * tire_dia)) =
           2*44.704/0.505 = 177.03 rad/s   -->
@@ -39,27 +39,22 @@
        axle_eff_limit = 204.95 / 2 N m = ~102.5 -->
   <!-- xacro:property name="axle_eff_limit" value="102.5"/ -->
-  <xacro:property name="axle_eff_limit" value="60"/>
+  <xacro:property name="axle_eff_limit" value="60" />
   <!-- max_speed = 33 Km/h = 9.17 m/s
        axle_vel_limit = (2 * pi) * (max_speed / (pi * tire_dia)) =  39.02 rad/s -->
-  <xacro:property name="axle_vel_limit" value="177.03"/>
+  <xacro:property name="axle_vel_limit" value="177.03" />
   <!-- Servo_stall_torque of the direction axis in Nm. servo_no_load_speed is
        measured in rad/s. -->
-  <xacro:property name="servo_stall_torque" value="50"/>  <!-- check -->
-  <xacro:property name="servo_no_load_speed" value="25"/> <!-- check -->
+  <xacro:property name="servo_stall_torque" value="50" /> <!-- check -->
+  <xacro:property name="servo_no_load_speed" value="25" /> <!-- check -->
   <!-- Inertia of a thick-walled cylindrical tube with open ends. Height is
        measured along the z axis, which is the tube's axis. inner_rad and
        outer_rad are the tube's inner and outer radii, respectively. -->
-  <xacro:macro name="thick_walled_tube_inertial"
-               params="inner_rad outer_rad height mass">
+  <xacro:macro name="thick_walled_tube_inertial" params="inner_rad outer_rad height mass">
     <inertial>
-      <mass value="${mass}"/>
+      <mass value="${mass}" />
       <inertia ixx="${(1 / 12) * mass * (3 * (inner_rad * inner_rad +
-                    outer_rad * outer_rad) + height * height)}"
-               ixy="0" ixz="0"
-               iyy="${(1 / 12) * mass * (3 * (inner_rad * inner_rad +
-                    outer_rad * outer_rad) + height * height)}"
-               iyz="0"
-               izz="${mass * (inner_rad * inner_rad +
-                    outer_rad * outer_rad) / 2}"/>
+                    outer_rad * outer_rad) + height * height)}" ixy="0" ixz="0" iyy="${(1 / 12) * mass * (3 * (inner_rad * inner_rad +
+                    outer_rad * outer_rad) + height * height)}" iyz="0" izz="${mass * (inner_rad * inner_rad +
+                    outer_rad * outer_rad) / 2}" />
     </inertial>
   </xacro:macro>
@@ -68,22 +63,20 @@
   <xacro:macro name="null_inertial">
     <inertial>
-      <mass value="0.001"/>
-      <inertia ixx="0.001" ixy="0" ixz="0" iyy="0.001" iyz="0" izz="0.001"/>
+      <mass value="0.001" />
+      <inertia ixx="0.001" ixy="0" ixz="0" iyy="0.001" iyz="0" izz="0.001" />
     </inertial>
   </xacro:macro>
   <!-- Shock absorber -->
-  <xacro:macro name="shock"
-               params="lr_prefix fr_prefix lr_reflect fr_reflect child">
+  <xacro:macro name="shock" params="lr_prefix fr_prefix lr_reflect fr_reflect child">
     <joint name="${lr_prefix}_${fr_prefix}_shock" type="prismatic">
-      <parent link="base_link"/>
-      <child link="${child}"/>
+      <parent link="base_link" />
+      <child link="${child}" />
       <origin xyz="${fr_reflect * wheelbase / 2}
                    ${lr_reflect * ((hex_hub_dist / 2) - axle_length)}
-                   ${-wheel_travel}"/>
-                  <!-- ${(wheel_travel / 2) - shock_z_offset}"/-->
-      <axis xyz="0 0 -1"/>
-      <limit lower="${-wheel_travel / 2}" upper="${wheel_travel / 2}"
-             effort="${shock_eff_limit}" velocity="${shock_vel_limit}"/>
-      <joint_properties damping="${suspension_joint_damping}" friction="{suspension_joint_friction}"/>
+                   ${-wheel_travel}" />
+      <!-- ${(wheel_travel / 2) - shock_z_offset}"/-->
+      <axis xyz="0 0 -1" />
+      <limit lower="${-wheel_travel / 2}" upper="${wheel_travel / 2}" effort="${shock_eff_limit}" velocity="${shock_vel_limit}" />
+      <joint_properties damping="${suspension_joint_damping}" friction="{suspension_joint_friction}" />
     </joint>
     <transmission name="${lr_prefix}_${fr_prefix}_shock_trans">
@@ -100,5 +93,5 @@
   <xacro:macro name="wheel" params="lr_prefix fr_prefix lr_reflect">
     <link name="${lr_prefix}_${fr_prefix}_axle_carrier">
-	  <!-- visual>
+      <!-- visual>
         <origin xyz="0 0 0"/>
         <geometry>
@@ -112,15 +105,15 @@
         </geometry>
 	  </collision -->
-      <xacro:null_inertial/>
+      <xacro:null_inertial />
     </link>
     <!-- The left and right axles have the same axis so that identical
          rotation values cause the wheels to rotate in the same direction. -->
     <joint name="${lr_prefix}_${fr_prefix}_axle" type="continuous">
-      <parent link="${lr_prefix}_${fr_prefix}_axle_carrier"/>
-      <child link="${lr_prefix}_${fr_prefix}_wheel"/>
-      <origin rpy="${degrees_90} 0 ${degrees_180}"/>
-      <axis xyz="0 0 -1"/>
-      <limit effort="${axle_eff_limit}" velocity="${axle_vel_limit}"/>
-      <joint_properties damping="${wheel_joint_damping}" friction="{wheel_joint_friction}"/>
+      <parent link="${lr_prefix}_${fr_prefix}_axle_carrier" />
+      <child link="${lr_prefix}_${fr_prefix}_wheel" />
+      <origin rpy="${degrees_90} 0 ${degrees_180}" />
+      <axis xyz="0 0 -1" />
+      <limit effort="${axle_eff_limit}" velocity="${axle_vel_limit}" />
+      <joint_properties damping="${wheel_joint_damping}" friction="{wheel_joint_friction}" />
     </joint>
     <transmission name="${lr_prefix}_${fr_prefix}_axle_trans">
@@ -141,21 +134,19 @@
         <origin xyz="0
                      0
-                     ${lr_reflect * (axle_length - (tire_width / 2 - hex_hub_depth))}"/>
-        <geometry>
-          <cylinder radius="${tire_dia / 2}" length="${tire_width}"/>
-        </geometry>
-        <material name="tire_mat"/>
+                     ${lr_reflect * (axle_length - (tire_width / 2 - hex_hub_depth))}" />
+        <geometry>
+          <cylinder radius="${tire_dia / 2}" length="${tire_width}" />
+        </geometry>
+        <material name="tire_mat" />
       </visual>
       <collision>
         <origin xyz="0
                      0
-                     ${lr_reflect * (axle_length - (tire_width / 2 - hex_hub_depth))}"/>
-        <geometry>
-          <cylinder radius="${tire_dia / 2}" length="${tire_width}"/>
+                     ${lr_reflect * (axle_length - (tire_width / 2 - hex_hub_depth))}" />
+        <geometry>
+          <cylinder radius="${tire_dia / 2}" length="${tire_width}" />
         </geometry>
       </collision>
-      <xacro:thick_walled_tube_inertial
-          inner_rad="${hub_dia / 2}" outer_rad="${tire_dia / 2}"
-          height="${tire_width}" mass="${wheel_mass}"/>
+      <xacro:thick_walled_tube_inertial inner_rad="${hub_dia / 2}" outer_rad="${tire_dia / 2}" height="${tire_width}" mass="${wheel_mass}" />
     </link>
     <gazebo reference="${lr_prefix}_${fr_prefix}_wheel">
@@ -165,11 +156,8 @@
   <!-- xacro:macro name="rubber_wheel" params="name parent *origin reflect hq" -->
   <!-- Front wheel -->
-  <xacro:macro name="front_wheel"
-               params="lr_prefix fr_prefix lr_reflect fr_reflect">
-    <xacro:shock lr_prefix="${lr_prefix}" fr_prefix="${fr_prefix}"
-                 lr_reflect="${lr_reflect}" fr_reflect="${fr_reflect}"
-                 child="${lr_prefix}_steering_link"/>
+  <xacro:macro name="front_wheel" params="lr_prefix fr_prefix lr_reflect fr_reflect">
+    <xacro:shock lr_prefix="${lr_prefix}" fr_prefix="${fr_prefix}" lr_reflect="${lr_reflect}" fr_reflect="${fr_reflect}" child="${lr_prefix}_steering_link" />
     <link name="${lr_prefix}_steering_link">
-	  <!-- visual>
+      <!-- visual>
 		<origin xyz="0 0 0"/>
         <geometry>
@@ -183,12 +171,11 @@
         </geometry>
 	  </collision -->
-      <xacro:null_inertial/>
+      <xacro:null_inertial />
     </link>
     <joint name="${lr_prefix}_steering_joint" type="revolute">
-      <parent link="${lr_prefix}_steering_link"/>
-      <child link="${lr_prefix}_${fr_prefix}_axle_carrier"/>
-      <axis xyz="0 0 1"/>
-      <limit lower="${-degrees_45}" upper="${degrees_45}"
-             effort="${servo_stall_torque}" velocity="${servo_no_load_speed}"/>
+      <parent link="${lr_prefix}_steering_link" />
+      <child link="${lr_prefix}_${fr_prefix}_axle_carrier" />
+      <axis xyz="0 0 1" />
+      <limit lower="${-degrees_45}" upper="${degrees_45}" effort="${servo_stall_torque}" velocity="${servo_no_load_speed}" />
     </joint>
     <transmission name="${lr_prefix}_steering_trans">
@@ -204,15 +191,10 @@
       <material>Gazebo/Black</material>
     </gazebo>
-    <xacro:wheel lr_prefix="${lr_prefix}" fr_prefix="${fr_prefix}"
-                 lr_reflect="${lr_reflect}"/>
+    <xacro:wheel lr_prefix="${lr_prefix}" fr_prefix="${fr_prefix}" lr_reflect="${lr_reflect}" />
   </xacro:macro>
   <!-- Rear wheel -->
-  <xacro:macro name="rear_wheel"
-               params="lr_prefix fr_prefix lr_reflect fr_reflect">
-    <xacro:shock lr_prefix="${lr_prefix}" fr_prefix="${fr_prefix}"
-                 lr_reflect="${lr_reflect}" fr_reflect="${fr_reflect}"
-                 child="${lr_prefix}_${fr_prefix}_axle_carrier"/>
-    <xacro:wheel lr_prefix="${lr_prefix}" fr_prefix="${fr_prefix}"
-                 lr_reflect="${lr_reflect}"/>
-  </xacro:macro>
- </robot>
+  <xacro:macro name="rear_wheel" params="lr_prefix fr_prefix lr_reflect fr_reflect">
+    <xacro:shock lr_prefix="${lr_prefix}" fr_prefix="${fr_prefix}" lr_reflect="${lr_reflect}" fr_reflect="${fr_reflect}" child="${lr_prefix}_${fr_prefix}_axle_carrier" />
+    <xacro:wheel lr_prefix="${lr_prefix}" fr_prefix="${fr_prefix}" lr_reflect="${lr_reflect}" />
+  </xacro:macro>
+</robot>
