Commit message: added basic model

File: description/urdf/perceus.xacro (robot description, xacro)
@@ -1,16 +1,26 @@
 <?xml version="1.0"?>
 <robot name="perceus">
+    <link name="dummy"></link>
     <link name="base_link">
         <inertial>
             <mass value="100.0" />
-            <origin xyz="0 0 0" />
+            <origin xyz="0 0 0" rpy="0 0 0" />
             <inertia ixx="1.391" ixy="0.004" ixz="0.0" iyy="6.853" iyz="0.0" izz="6.125" />
         </inertial>
         <visual>
-            <origin xyz="0 0 0"/>
+            <origin xyz="0 0 0.5" rpy="0 0 0" />
             <geometry>
-                <box length="2.0" width="2.0" height="1.0"/>
+                <box size="2.0 2.0 1.0" />
             </geometry>
         </visual>
+        <collision>
+            <geometry>
+                <box size="3 3 2" />
+            </geometry>
+        </collision>
     </link>
+    <joint name="dummy_joint" type="fixed">
+        <parent link="dummy" />
+        <child link="base_link" />
+    </joint>
 </robot>

Commit message: basic urdf made

File: description/urdf/perceus.xacro (robot description, xacro)
@@ -1,26 +1,107 @@
 <?xml version="1.0"?>
-<robot name="perceus">
-    <link name="dummy"></link>
-    <link name="base_link">
-        <inertial>
-            <mass value="100.0" />
-            <origin xyz="0 0 0" rpy="0 0 0" />
-            <inertia ixx="1.391" ixy="0.004" ixz="0.0" iyy="6.853" iyz="0.0" izz="6.125" />
-        </inertial>
-        <visual>
-            <origin xyz="0 0 0.5" rpy="0 0 0" />
-            <geometry>
-                <box size="2.0 2.0 1.0" />
-            </geometry>
-        </visual>
-        <collision>
-            <geometry>
-                <box size="3 3 2" />
-            </geometry>
-        </collision>
-    </link>
-    <joint name="dummy_joint" type="fixed">
-        <parent link="dummy" />
-        <child link="base_link" />
-    </joint>
+<!-- A simple model of the racecar for rviz -->
+<robot xmlns:xacro="http://www.ros.org/wiki/xacro" name="racecar">
+  <xacro:property name="wheelbase" value="0.3302" />
+  <xacro:property name="width" value="0.2032" />
+  <xacro:property name="height" value="0.1" />
+  <xacro:property name="ground_offset" value="0.04" />
+  <xacro:property name="wheel_radius" value="0.0508" />
+  <xacro:property name="wheel_length" value="0.0381" />
+  <xacro:property name="laser_distance_from_base_link" value="0.275" />
+  <xacro:property name="laser_height" value="0.05" />
+  <xacro:property name="laser_radius" value="0.026" />
+  <material name="black">
+    <color rgba="0.2 0.2 0.2 1.0"/>
+  </material>
+  <material name="blue">
+    <color rgba="0.3 0.57 1. 1.0"/>
+  </material>
+  <link name="base_link">
+    <visual>
+      <origin xyz="${wheelbase/2} 0 ${ground_offset+height/2}"/>
+      <geometry>
+        <box size="${wheelbase} ${width} ${height}"/>
+      </geometry>
+      <material name="blue"/>
+    </visual>
+  </link>
+  <joint name="base_to_laser_model" type="fixed">
+    <parent link="base_link"/>
+    <child link="laser_model"/>
+    <origin xyz="${laser_distance_from_base_link} 0 ${ground_offset+height+(laser_height/2)}"/>
+  </joint>
+  <link name="laser_model">
+    <visual>
+      <geometry>
+        <cylinder radius="${laser_radius}" length="${laser_height}"/>
+      </geometry>
+      <material name="black"/>
+    </visual>
+  </link>
+  <joint name="base_to_back_left_wheel" type="fixed">
+    <parent link="base_link"/>
+    <child link="back_left_wheel"/>
+    <origin xyz="0 ${(wheel_length+width)/2} ${wheel_radius}"/>
+  </joint>
+  <link name="back_left_wheel">
+    <visual>
+      <geometry>
+        <cylinder radius="${wheel_radius}" length="${wheel_length}"/>
+      </geometry>
+      <material name="black"/>
+      <origin rpy="${pi/2} 0 0"/>
+    </visual>
+  </link>
+  <joint name="base_to_back_right_wheel" type="fixed">
+    <parent link="base_link"/>
+    <child link="back_right_wheel"/>
+    <origin xyz="0 ${-(wheel_length+width)/2} ${wheel_radius}"/>
+  </joint>
+  <link name="back_right_wheel">
+    <visual>
+      <geometry>
+        <cylinder radius="${wheel_radius}" length="${wheel_length}"/>
+      </geometry>
+      <material name="black"/>
+      <origin rpy="${pi/2} 0 0"/>
+    </visual>
+  </link>
+  <joint name="base_to_front_left_hinge" type="fixed">
+    <parent link="base_link"/>
+    <child link="front_left_hinge"/>
+    <origin xyz="${wheelbase} ${(wheel_length+width)/2} ${wheel_radius}"/>
+  </joint>
+  <link name="front_left_hinge"/>
+  <joint name="front_left_hinge_to_wheel" type="continuous">
+    <parent link="front_left_hinge"/>
+    <child link="front_left_wheel"/>
+  </joint>
+  <link name="front_left_wheel">
+    <visual>
+      <geometry>
+        <cylinder radius="${wheel_radius}" length="${wheel_length}"/>
+      </geometry>
+      <material name="black"/>
+      <origin rpy="${pi/2} 0 0"/>
+    </visual>
+  </link>
+  <joint name="base_to_front_right_hinge" type="fixed">
+    <parent link="base_link"/>
+    <child link="front_right_hinge"/>
+    <origin xyz="${wheelbase} ${-(wheel_length+width)/2} ${wheel_radius}"/>
+  </joint>
+  <link name="front_right_hinge"/>
+  <joint name="front_right_hinge_to_wheel" type="continuous">
+    <parent link="front_right_hinge"/>
+    <child link="front_right_wheel"/>
+  </joint>
+  <link name="front_right_wheel">
+    <visual>
+      <geometry>
+        <cylinder radius="${wheel_radius}" length="${wheel_length}"/>
+      </geometry>
+      <material name="black"/>
+      <origin rpy="${pi/2} 0 0"/>
+    </visual>
+  </link>
 </robot>
