Commit message: made lidar parallel to ground

File: eufs_description/robots/ads-dv.urdf.xacro (robot description, xacro)
@@ -60,5 +60,5 @@
     </xacro:VLP-16> -->
     <xacro:VLP-16R  parent="base_link" name="velodyne" topic="/velodyne_points" hz="10" samples="800">
-        <origin xyz="1.58 0.0 -0.1" rpy="0 ${1*M_PI/180.0} 0"/>
+        <origin xyz="1.58 0.0 -0.1" rpy="0 0 0"/>
     </xacro:VLP-16R>
     <xacro:zed_camera parent="base_link" prefix="zed">

Commit message: added sick_lms_1xx

File: eufs_description/robots/ads-dv.urdf.xacro (robot description, xacro)
@@ -52,4 +52,7 @@
         <origin xyz="1.700 0.0 -0.080" rpy="0 -0.0174533 0"/>
     </xacro:sensor_hokuyo_utm30lx> -->
+    <xacro:sick_lms1xx parent="base_link" prefix="lidar">
+        <origin xyz="1.700 0.0 -0.080" rpy="0 -0.0174533 0" />
+    </xacro:sick_lms1xx>
     <!-- <xacro:VLP-16  parent="base_link" name="velodyne" topic="/velodyne_points" hz="10">
         <origin xyz="1.700 0.0 -0.150" rpy="0 -0.0174533 0"/>

File: eufs_description/sensors/all_sensors.urdf.xacro (robot description, xacro)
@@ -6,4 +6,6 @@
   <!-- Hokuyo utm30lx -->
   <xacro:include filename="$(find eufs_description)/sensors/hokuyo_utm30lx.urdf.xacro" />
+  <!-- SICK LMS 1xx -->
+  <xacro:include filename="$(find eufs_description)/sensors/sick_lms1xx.urdf.xacro" />
   <!-- Velodyne VLP-16 -->
   <xacro:include filename="$(find eufs_description)/sensors/VLP-16.urdf.xacro" />

Commit message: switched to 2d lidar | removed redundancies

File: eufs_description/robots/ads-dv.urdf.xacro (robot description, xacro)
@@ -53,5 +53,5 @@
     </xacro:sensor_hokuyo_utm30lx> -->
     <xacro:sick_lms1xx parent="base_link" prefix="lidar">
-        <origin xyz="1.700 0.0 -0.080" rpy="0 -0.0174533 0" />
+        <origin xyz="1.700 0.0 -0.080" rpy="0 -0 0" />
     </xacro:sick_lms1xx>
     <!-- <xacro:VLP-16  parent="base_link" name="velodyne" topic="/velodyne_points" hz="10">

File: eufs_description/sensors/sick_lms1xx.urdf.xacro (robot description, xacro)
@@ -1,5 +1,5 @@
 <?xml version="1.0"?>
 <robot xmlns:xacro="http://www.ros.org/wiki/xacro">
-    <xacro:macro name="sick_lms1xx" params="parent:=base_link prefix:=eufs *origin frame:=laser topic:=scan sample_size:=720 update_rate:=50 min_angle:=-2.35619 max_angle:=2.35619 min_range:=0.1 max_range:=30.0 robot_namespace:=/">
+    <xacro:macro name="sick_lms1xx" params="parent:=base_link prefix:=eufs *origin frame:=laser topic:=scan sample_size:=720 update_rate:=50 min_angle:=-1.57 max_angle:=1.57 min_range:=0.1 max_range:=10.0 robot_namespace:=/">
         <joint name="${prefix}_base_joint" type="fixed">
             <!-- FRONT MOUNT  -->
@@ -35,5 +35,5 @@
             <sensor type="ray" name="${frame}">
                 <pose>0 0 0 0 0 0</pose>
-                <visualize>false</visualize>
+                <visualize>true</visualize>
                 <update_rate>${update_rate}</update_rate>
                 <ray>
