Commit message: added dynamic origin

File: eufs_description/sensors/sick_lms1xx.urdf.xacro (robot description, xacro)
@@ -1,5 +1,5 @@
 <?xml version="1.0"?>
 <robot xmlns:xacro="http://www.ros.org/wiki/xacro">
-    <xacro:macro name="sick_lms1xx" params="frame:=laser topic:=scan sample_size:=720 update_rate:=50 min_angle:=-2.35619 max_angle:=2.35619 min_range:=0.1 max_range:=30.0 robot_namespace:=/">
+    <xacro:macro name="sick_lms1xx" params="parent:=base_link prefix:=eufs *origin frame:=laser topic:=scan sample_size:=720 update_rate:=50 min_angle:=-2.35619 max_angle:=2.35619 min_range:=0.1 max_range:=30.0 robot_namespace:=/">
         <joint name="${prefix}_base_joint" type="fixed">
             <!-- FRONT MOUNT  -->
@@ -11,5 +11,5 @@
             <child link="${prefix}_base_link" />
         </joint>
-        <link name="${frame}">
+        <link name="${prefix}_base_link">
             <inertial>
                 <mass value="1.1" />
